Commit message: Ros2 Mechanum Controller added.

File: src/ecza_description/urdf/rover.urdf.xacro (robot description, xacro)
@@ -168,3 +168,41 @@
     <origin xyz="0 0 ${chassis_height}" rpy="0 0 0"/>
   </joint>
+  <!-- ── ros2_control — topic_based hardware interface ─────────────────── -->
+  <!--
+    topic_based_ros2_control bridges joint velocity commands and states via
+    ROS topics, connecting mecanum_drive_controller to the ESP32 micro-ROS.
+    Command topic : /wheel_velocities_cmd  (std_msgs/Float32MultiArray)
+      data = [fl, fr, rl, rr] rad/s  (written by mecanum_drive_controller)
+    State topic   : /wheel_velocities      (std_msgs/Float32MultiArray)
+      data = [fl, fr, rl, rr] rad/s  (published by ESP32 micro-ROS)
+    Joint order must match the array index order used in velocity_subscriber.c:
+      0=fl  1=fr  2=rl  3=rr
+  -->
+  <ros2_control name="ecza_rover_hardware" type="system">
+    <hardware>
+      <plugin>topic_based_ros2_control/TopicBasedSystem</plugin>
+      <param name="joint_commands_topic">/wheel_velocities_cmd</param>
+      <param name="joint_states_topic">/wheel_velocities</param>
+    </hardware>
+    <joint name="fl_wheel_joint">
+      <command_interface name="velocity"/>
+      <state_interface name="velocity"/>
+      <state_interface name="position"/>
+    </joint>
+    <joint name="fr_wheel_joint">
+      <command_interface name="velocity"/>
+      <state_interface name="velocity"/>
+      <state_interface name="position"/>
+    </joint>
+    <joint name="rl_wheel_joint">
+      <command_interface name="velocity"/>
+      <state_interface name="velocity"/>
+      <state_interface name="position"/>
+    </joint>
+    <joint name="rr_wheel_joint">
+      <command_interface name="velocity"/>
+      <state_interface name="velocity"/>
+      <state_interface name="position"/>
+    </joint>
+  </ros2_control>
 </robot>

Commit message: fix(nav2): fix bt_navigator plugins, SLAM TF timeout, RViz Nav2 goal tool

File: src/ecza_description/urdf/rover.urdf.xacro (robot description, xacro)
@@ -168,4 +168,35 @@
     <origin xyz="0 0 ${chassis_height}" rpy="0 0 0"/>
   </joint>
+  <!-- ── RPLidar A2M12 ─────────────────────────────────────────────────── -->
+  <!--
+    Mounted on top of the chassis, centred, facing forward.
+    Height: chassis top (chassis_z + ch2) + 30 mm standoff + ~15 mm sensor half-height.
+    The laser plane is horizontal at the top of the sensor body.
+    Frame: laser_frame  (REP-105 sensor frame, Z up, X forward)
+  -->
+  <link name="laser_frame">
+    <visual>
+      <geometry>
+        <cylinder radius="0.038" length="0.060"/>
+      </geometry>
+      <material name="chassis_grey"/>
+    </visual>
+    <collision>
+      <geometry>
+        <cylinder radius="0.038" length="0.060"/>
+      </geometry>
+    </collision>
+    <xacro:cylinder_inertia m="0.17" r="0.038" h="0.060"/>
+  </link>
+  <joint name="laser_joint" type="fixed">
+    <parent link="base_link"/>
+    <child  link="laser_frame"/>
+    <!--
+      x=0 : centred front-back
+      y=0 : centred left-right
+      z   : top of chassis + 15 mm standoff + 30 mm to laser plane
+    -->
+    <origin xyz="0.0 0.0 ${chassis_z + ch2 + 0.045}" rpy="0 0 0"/>
+  </joint>
   <!-- ── ros2_control — topic_based hardware interface ─────────────────── -->
   <!--

Commit message: hasan devraldı

File: src/ecza_description/urdf/rover.urdf.xacro (robot description, xacro)
@@ -8,5 +8,5 @@
     wheel_separation_width : 0.26 m   (left/right centre-to-centre)
     wheel_base             : 0.38 m   (front/rear axle centre-to-centre)
-    wheel_radius           : 0.05 m   (placeholder — update when measured)
+    wheel_radius           : 0.08 m   (measured physical wheel)
   Frame convention (ROS REP-103):
     base_link  — geometric centre of chassis, mid-height
@@ -20,5 +20,5 @@
   <xacro:property name="chassis_height"    value="0.08"/>
   <xacro:property name="chassis_mass"      value="3.0"/>   <!-- kg, estimate -->
-  <xacro:property name="wheel_radius"      value="0.05"/>
+  <xacro:property name="wheel_radius"      value="0.08"/>  <!-- must match rover_params.yaml and controllers.yaml -->
   <xacro:property name="wheel_width"       value="0.03"/>
   <xacro:property name="wheel_mass"        value="0.15"/>
@@ -111,5 +111,5 @@
       indicate the 45° passive roller direction — purely cosmetic in URDF.
   -->
-  <xacro:macro name="mecanum_wheel" params="name x_pos y_pos roller_angle">
+  <xacro:macro name="mecanum_wheel" params="name x_pos y_pos roller_angle axis_y">
     <link name="${name}_wheel_link">
       <!-- Main wheel drum -->
@@ -149,5 +149,5 @@
       <child  link="${name}_wheel_link"/>
       <origin xyz="${x_pos} ${y_pos} 0" rpy="0 0 0"/>
-      <axis xyz="0 1 0"/>
+      <axis xyz="0 ${axis_y} 0"/>
       <dynamics damping="0.01" friction="0.1"/>
     </joint>
@@ -157,8 +157,11 @@
        FR/RL: roller_angle = -pi/4  (\ rollers)
   -->
-  <xacro:mecanum_wheel name="fl" x_pos=" ${cl2}" y_pos=" ${cw2 + wheel_width/2}" roller_angle=" ${pi/4}"/>
-  <xacro:mecanum_wheel name="fr" x_pos=" ${cl2}" y_pos="-${cw2 + wheel_width/2}" roller_angle="-${pi/4}"/>
-  <xacro:mecanum_wheel name="rl" x_pos="-${cl2}" y_pos=" ${cw2 + wheel_width/2}" roller_angle="-${pi/4}"/>
-  <xacro:mecanum_wheel name="rr" x_pos="-${cl2}" y_pos="-${cw2 + wheel_width/2}" roller_angle=" ${pi/4}"/>
+  <!-- axis_y: left wheels use +1 (outward = +Y), right wheels use -1 (outward = -Y).
+       This ensures positive joint velocity = robot-forward for all wheels,
+       matching the firmware's raw pass-through (no per-wheel sign correction). -->
+  <xacro:mecanum_wheel name="fl" x_pos=" ${cl2}" y_pos=" ${cw2 + wheel_width/2}" roller_angle=" ${pi/4}" axis_y= "1"/>
+  <xacro:mecanum_wheel name="fr" x_pos=" ${cl2}" y_pos="-${cw2 + wheel_width/2}" roller_angle="-${pi/4}" axis_y="-1"/>
+  <xacro:mecanum_wheel name="rl" x_pos="-${cl2}" y_pos=" ${cw2 + wheel_width/2}" roller_angle="-${pi/4}" axis_y= "1"/>
+  <xacro:mecanum_wheel name="rr" x_pos="-${cl2}" y_pos="-${cw2 + wheel_width/2}" roller_angle=" ${pi/4}" axis_y="-1"/>
   <!-- ── IMU frame (centred on chassis top) ─────────────────────────────── -->
   <link name="imu_link"/>

Commit message: otonom gitmeye başladı

File: src/ecza_description/urdf/rover.urdf.xacro (robot description, xacro)
@@ -200,5 +200,5 @@
       z   : top of chassis + 15 mm standoff + 30 mm to laser plane
     -->
-    <origin xyz="0.0 0.0 ${chassis_z + ch2 + 0.045}" rpy="0 0 0"/>
+    <origin xyz="0.0 0.0 ${chassis_z + ch2 + 0.045}" rpy="0 0 3.14159"/>
   </joint>
   <!-- ── ros2_control — topic_based hardware interface ─────────────────── -->
